File: OPENpsu30.kicad_pcb (KiCad board)
At the start: 2 copper layers, 188 x 108.5 mm, 18 parts, among them J1 output, J2 Conn_01x04_Pin APPL, J3 Conn_01x03_Socket astec?, J4 Conn_01x01_Pin_sony_pos, J5 Conn_01x01_Pin_sony_NEG

Commit message: upd
Other:
- board text added: "V 0.011"
- board text removed: "V 0.01"
Changed lines of the file:
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@@
 		)
 	)
-	(gr_text "V 0.01"
+	(gr_text "V 0.011\n"
 		(at 84.5 112 0)
 		(layer "F.SilkS")
@@
 			(justify left bottom)
 		)
-		(render_cache "V 0.01" 0
+		(render_cache "V 0.011\n" 0
 			(polygon
 				(pts
@@
 				)
 			)
+			(polygon
+				(pts
+					(xy 104.007676 107.318325) (xy 103.175785 111.32) (xy 102.334124 111.32) (xy 102.964026 108.290167)
+					(xy 102.774738 108.408869) (xy 102.551988 108.509986) (xy 102.31434 108.586434) (xy 102.077913 108.631374)
+					(xy 102.230565 107.896692) (xy 102.57348 107.786108) (xy 102.901988 107.649274) (xy 103.215495 107.489375)
+					(xy 103.497208 107.318325)
+				)
+			)

Commit message: upd ver
Other:
- board text added: "V 0.012"
- board text removed: "V 0.011"
Changed lines of the file:
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@@
 		)
 	)
-	(gr_text "V 0.011\n"
+	(gr_text "V 0.012\n"
 		(at 84.5 112 0)
 		(layer "F.SilkS")
@@
 			(justify left bottom)
 		)
-		(render_cache "V 0.011\n" 0
+		(render_cache "V 0.012\n" 0
 			(polygon
 				(pts
@@
 			(polygon
 				(pts
-					(xy 104.007676 107.318325) (xy 103.175785 111.32) (xy 102.334124 111.32) (xy 102.964026 108.290167)
-					(xy 102.774738 108.408869) (xy 102.551988 108.509986) (xy 102.31434 108.586434) (xy 102.077913 108.631374)
-					(xy 102.230565 107.896692) (xy 102.57348 107.786108) (xy 102.901988 107.649274) (xy 103.215495 107.489375)
-					(xy 103.497208 107.318325)
+					(xy 102.24815 110.600949) (xy 103.873098 110.600949) (xy 103.723621 111.32) (xy 101.174214 111.32)
+					(xy 101.236252 111.021779) (xy 101.321209 110.734136) (xy 101.447034 110.482979) (xy 101.60687 110.255155)
+					(xy 101.784822 110.054577) (xy 101.979843 109.874651) (xy 102.181716 109.718743) (xy 102.574703 109.45545)
+					(xy 102.918841 109.220488) (xy 103.178715 108.997739) (xy 103.279695 108.883769) (xy 103.355059 108.773524)
+					(xy 103.411615 108.65619) (xy 103.44836 108.531479) (xy 103.464646 108.365649) (xy 103.442289 108.242838)
+					(xy 103.388276 108.150704) (xy 103.303788 108.084076) (xy 103.176536 108.039086) (xy 102.99016 108.021744)
+					(xy 102.753576 108.044542) (xy 102.505828 108.11541) (xy 102.242613 108.240353) (xy 101.959944 108.428164)
+					(xy 102.118213 107.665882) (xy 102.410131 107.519053) (xy 102.705384 107.415973) (xy 103.006231 107.354517)
+					(xy 103.315247 107.333956) (xy 103.59518 107.354664) (xy 103.821318 107.41187) (xy 104.018722 107.508768)
+					(xy 104.166678 107.634619) (xy 104.273807 107.793155) (xy 104.338136 107.98584) (xy 104.356041 108.198076)
+					(xy 104.326657 108.446482) (xy 104.25179 108.705642) (xy 104.14494 108.927641) (xy 104.008055 109.128812)
+					(xy 103.848674 109.310369) (xy 103.669896 109.474744) (xy 103.471807 109.626175) (xy 103.048046 109.903635)
+					(xy 102.762526 110.08755) (xy 102.515352 110.267313) (xy 102.335101 110.440237) (xy 102.275873 110.526327)
 				)
 			)
