File: OPENpsu30.kicad_pcb (KiCad board)
At the start: 2 copper layers, 188 x 108.5 mm, 18 parts, among them J1 output, J2 Conn_01x04_Pin APPL, J3 Conn_01x03_Socket astec?, J4 Conn_01x01_Pin_sony_pos, J5 Conn_01x01_Pin_sony_NEG

Commit message: test
Parts:
- removed REF**: MountingHole_3.5mm_Pad, MountingHole:MountingHole_3.5mm_Pad
- added ?: , , F.Cu at (91.5, 51.5)
- added G***: LOGO, LOGO, F.Cu at (90.5, 125.0)
- added G***: LOGO, LOGO, B.Cu at (210.5, 56.0)
- added J6: Conn_01x01_Pin_sony_pos, Library:pin 1.65, F.Cu at (256.0, 88.0)
- J3: footprint TerminalBlock:TerminalBlock_MaiXu_MX126-5.0-03P_1x03_P5.00mm -> Connector_Phoenix_MSTB:PhoenixContact_MSTBVA_2,5_3-G-5,08_1x03_P5.08mm_Vertical
- J4, J5: footprint Connector_Samtec_HPM_THT:Samtec_HPM-01-01-x-S_Straight_1x01_Pitch5.08mm -> Library:pin 1.65
Other:
- board text added: "120/240V AC"
- board text added: "V 0.020"
- board text added: "github.com/Toucan45/Open-Mac-Psu/"
- board text removed: "2"
- board text removed: "T"
- board text removed: "V 0.012"

Commit message: upd ver #
Other:
- board text added: "V 0.031"
- board text removed: "V 0.020"

Commit message: Add files via upload
Parts:
- renumbered G*** to f
Other:
- board text added: "2can.top"
- board text added: "V 1.1"
- board text removed: "V 0.031"

Commit message: Add files via upload
Routing:
- net (no net): track 0.00 -> 22.5 mm
Other:
- board text added: "V 1.2"
- board text removed: "V 1.1"
Changed lines of the file:
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@@
 		(embedded_fonts no)
 	)
+	(gr_poly
+		(pts
+			(xy 79.5 62) (xy 79.5 51) (xy 86.5 51) (xy 92 47) (xy 96.5 47) (xy 96.5 56.5) (xy 86 62)
+		)
+		(stroke
+			(width 0.2)
+			(type solid)
+		)
+		(fill yes)
+		(layer "B.Cu")
+		(net 1)
+	)
+	(gr_rect
+		(start 161 50.5)
+		(end 171.5 68.5)
+		(stroke
+			(width 0.2)
+			(type solid)
+		)
+		(fill yes)
+		(layer "B.Cu")
+		(net 1)
+	)
 	(gr_rect
 		(start 253.5 76.5)
@@
 		)
 	)
-	(gr_text "V 1.1\n"
+	(gr_text "V 1.2\n"
 		(at 82.5 114 0)
 		(layer "F.SilkS")
@@
 			(justify left bottom)
 		)
-		(render_cache "V 1.1\n" 0
+		(render_cache "V 1.2\n" 0
 			(polygon
 				(pts
@@
 			(polygon
 				(pts
-					(xy 95.56748 109.318325) (xy 94.735589 113.32) (xy 93.893928 113.32) (xy 94.523831 110.290167)
-					(xy 94.334542 110.408869) (xy 94.111793 110.509986) (xy 93.874145 110.586434) (xy 93.637718 110.631374)
-					(xy 93.790369 109.896692) (xy 94.133285 109.786108) (xy 94.461793 109.649274) (xy 94.7753 109.489375)
-					(xy 95.057013 109.318325)
+					(xy 93.807955 112.600949) (xy 95.432903 112.600949) (xy 95.283426 113.32) (xy 92.734019 113.32)
+					(xy 92.796057 113.021779) (xy 92.881013 112.734136) (xy 93.006838 112.482979) (xy 93.166674 112.255155)
+					(xy 93.344626 112.054577) (xy 93.539648 111.874651) (xy 93.741521 111.718743) (xy 94.134508 111.45545)
+					(xy 94.478646 111.220488) (xy 94.73852 110.997739) (xy 94.8395 110.883769) (xy 94.914863 110.773524)
+					(xy 94.97142 110.65619) (xy 95.008164 110.531479) (xy 95.024451 110.365649) (xy 95.002093 110.242838)
+					(xy 94.94808 110.150704) (xy 94.863593 110.084076) (xy 94.736341 110.039086) (xy 94.549965 110.021744)
+					(xy 94.313381 110.044542) (xy 94.065632 110.11541) (xy 93.802418 110.240353) (xy 93.519748 110.428164)
+					(xy 93.678018 109.665882) (xy 93.969935 109.519053) (xy 94.265188 109.415973) (xy 94.566036 109.354517)
+					(xy 94.875052 109.333956) (xy 95.154985 109.354664) (xy 95.381123 109.41187) (xy 95.578527 109.508768)
+					(xy 95.726482 109.634619) (xy 95.833611 109.793155) (xy 95.897941 109.98584) (xy 95.915846 110.198076)
+					(xy 95.886461 110.446482) (xy 95.811595 110.705642) (xy 95.704745 110.927641) (xy 95.567859 111.128812)
+					(xy 95.408478 111.310369) (xy 95.229701 111.474744) (xy 95.031612 111.626175) (xy 94.60785 111.903635)
+					(xy 94.32233 112.08755) (xy 94.075157 112.267313) (xy 93.894905 112.440237) (xy 93.835677 112.526327)
 				)
 			)
@@
 	)
 	(segment
+		(start 261.5 31.5)
+		(end 239 31.5)
+		(width 4)
+		(layer "B.Cu")
+		(net 0)
+	)
+	(segment
